Commit message: Migration to ROS2, fixes

File: urdf/kinect.urdf.xacro (robot description, xacro)
@@ -1,94 +1,92 @@
 <?xml version="1.0"?>
 <robot name="sensor" xmlns:xacro="http://www.ros.org/wiki/xacro">
-      <xacro:property name="height1" value="1.2" />
-  <xacro:property name="height2" value="0.5" />
-  <xacro:property name="width" value="0.2" />
-  <xacro:property name="mass" value="0.1" />
- <!-- Used for fixing robot to Gazebo 'base_link' -->
-  <link name="world"/>
-  <joint name="fixed" type="fixed">
-    <parent link="world"/>
-    <child link="kinect_link"/>
-    <origin xyz="0 0 0.1" rpy="0 0 0"/>
-  </joint>
-  <!-- Kinect Link -->
-  <link name="kinect_link">
-    <collision>
-      <origin xyz="0 0 0.1" rpy="0 0 0"/>
-      <geometry>
-	<mesh filename="$(find sensors_demos_gazebo)/meshes/kinect.dae" scale="0.001 0.001 0.001" />
-      </geometry>
-    </collision>
-    <visual>
-      <origin xyz="0 0 0.1" rpy="0 0 0"/>
-      <geometry>
-         <mesh filename="$(find sensors_demos_gazebo)/meshes/kinect.dae" scale="0.001 0.001 0.001" />
-      </geometry>
-      <material name="orange"/>
-    </visual>
-    <inertial>
-      <origin xyz="0 0 0" rpy="0 0 0"/>
-      <mass value="${mass}"/>
-      <inertia
-	  ixx="${mass}" ixy="0.0" ixz="0.0"
-	  iyy="${mass}" iyz="0.0"
-	  izz="${mass}"/>
-    </inertial>
-  </link>
-  <link name="kinect_optical_link">
-<!--      <visual>
-      <origin xyz="0 0 0" rpy="0 0 0"/>
-      <geometry>
-        <box size="0.01 0.01 0.01"/>
-      </geometry>
-      <material name="orange"/>
-    </visual>-->
-  </link>
-  <joint name="optical_joint" type="fixed">
-    <parent link="kinect_link"/>
-    <child link="kinect_optical_link"/>
-    <origin xyz="0.01 0 0.15" rpy="0.0 0 0"/>
-  </joint>
-  <material name="orange">
-    <color rgba="${255/255} ${108/255} ${10/255} 1.0"/>
-  </material>
-    <gazebo reference="kinect_optical_link">
-    <sensor type="depth" name="kinect_depth_sensor">
-        <always_on>0</always_on>
-	<update_rate>1</update_rate>
-        <horizontal_fov> ${91.2*3.14/180} </horizontal_fov>
-        <vertical_fov> ${65.5*3.14/180} </vertical_fov>
-        <diagonal_fov> ${100.6*3.14/180} </diagonal_fov>
-        <camera name="kinect">
-          <image>
-            <format>R8G8B8</format>
-            <width>640</width>
-            <height>480</height>
-          </image>
-          <clip>
-            <near>0.05</near>
-            <far>4.0</far>
-          </clip>
-          <noise>
-            <type>gaussian</type>
-            <mean>0.0</mean>
-            <stddev>0.005</stddev>
-          </noise>
-        </camera>
-        <plugin name="kinect_frame_controller" filename="libgazebo_ros_camera.so">
-	   <camera_name>kinect</camera_name>
-          <alwaysOn>true</alwaysOn>
-          <updateRate>6.0</updateRate>
-          <cameraName>kinect</cameraName>
-          <imageTopicName>color/image_raw</imageTopicName>
-          <depthImageTopicName>depth/image_rect_raw</depthImageTopicName>
-          <cameraInfoTopicName>color/camera_info</cameraInfoTopicName>
-          <depthImageCameraInfoTopicName>depth/camera_info</depthImageCameraInfoTopicName>
-          <pointCloudTopicName>depth_registered/points</pointCloudTopicName>
-          <frameName>kinect_link</frameName>
-          <pointCloudCutoff>0.05</pointCloudCutoff>
-          <rangeMax>8.0</rangeMax>
-        </plugin>
-	</sensor>
+    <xacro:property name="sensor_name" value="kinect" />
+    <xacro:property name="height1" value="1.2" />
+    <xacro:property name="height2" value="0.5" />
+    <xacro:property name="width" value="0.2" />
+    <xacro:property name="mass" value="0.1" />
+    <!-- Used for fixing robot to Gazebo 'base_link' -->
+    <link name="world"/>
+    <joint name="fixed" type="fixed">
+        <parent link="world"/>
+        <child link="${sensor_name}_link"/>
+        <origin xyz="0 0 0.1" rpy="0 0 0"/>
+    </joint>
+    <!-- Kinect Link -->
+    <link name="${sensor_name}_link">
+        <collision>
+            <origin xyz="0 0 0.1" rpy="0 0 0"/>
+            <geometry>
+                <mesh filename="$(find sensors_demos_gazebo)/meshes/kinect.dae" scale="0.001 0.001 0.001" />
+            </geometry>
+        </collision>
+        <visual>
+            <origin xyz="0 0 0.1" rpy="0 0 0"/>
+            <geometry>
+                <mesh filename="$(find sensors_demos_gazebo)/meshes/kinect.dae" scale="0.001 0.001 0.001" />
+            </geometry>
+            <material name="orange"/>
+        </visual>
+        <inertial>
+            <origin xyz="0 0 0" rpy="0 0 0"/>
+            <mass value="${mass}"/>
+            <inertia ixx="${mass}" ixy="0.0" ixz="0.0" iyy="${mass}" iyz="0.0" izz="${mass}"/>
+        </inertial>
+    </link>
+    <link name="${sensor_name}_optical_link">
+    <!--<visual>
+            <origin xyz="0 0 0" rpy="0 0 0"/>
+            <geometry>
+                <box size="0.01 0.01 0.01"/>
+            </geometry>
+            <material name="orange"/>
+        </visual>-->
+    </link>
+    <joint name="optical_joint" type="fixed">
+        <parent link="${sensor_name}_link"/>
+        <child link="${sensor_name}_optical_link"/>
+        <origin xyz="0.01 0 0.15" rpy="0.0 0 0"/>
+    </joint>
+    <material name="orange">
+        <color rgba="${255/255} ${108/255} ${10/255} 1.0"/>
+    </material>
+    <gazebo reference="${sensor_name}_optical_link">
+        <sensor type="depth" name="${sensor_name}_depth_sensor">
+            <always_on>0</always_on>
+            <update_rate>1</update_rate>
+            <camera name="${sensor_name}">
+                <horizontal_fov> ${91.2*3.14/180} </horizontal_fov>
+                <vertical_fov> ${65.5*3.14/180} </vertical_fov>
+                <diagonal_fov> ${100.6*3.14/180} </diagonal_fov>
+                <image>
+                    <format>R8G8B8</format>
+                    <width>640</width>
+                    <height>480</height>
+                </image>
+                <clip>
+                    <near>0.05</near>
+                    <far>4.0</far>
+                </clip>
+                <noise>
+                    <type>gaussian</type>
+                    <mean>0.0</mean>
+                    <stddev>0.005</stddev>
+                </noise>
+            </camera>
+            <plugin name="${sensor_name}_frame_controller" filename="libgazebo_ros_camera.so">
+                <ros>
+                    <namespace>${sensor_name}</namespace>
+                    <remapping>${sensor_name}/image_raw:=color/image_raw</remapping>
+                    <remapping>${sensor_name}/depth/image_raw:=depth/image_rect_raw</remapping>
+                    <remapping>${sensor_name}/camera_info:=camera_info</remapping>
+                    <remapping>${sensor_name}/depth/camera_info:=depth/camera_info</remapping>
+                    <remapping>${sensor_name}/points:=depth/points</remapping>
+                </ros>
+                <camera_name>${sensor_name}</camera_name>
+                <frame_name>${sensor_name}_link</frame_name>
+                <min_depth>0.05</min_depth>
+                <max_depth>8.0</max_depth>
+            </plugin>
+	    </sensor>
 	</gazebo>
 </robot>
