Commit message: Added another sensors

File: urdf/hokuyo.urdf.xacro (robot description, xacro)
@@ -17,5 +17,5 @@
       <origin xyz="0 0 0.0" rpy="1.57 0 0"/>
       <geometry>
-          <mesh filename="package://sensors_demos_gazebo/meshes/utm30.dae" scale="1 1 1"/>
+	  <mesh filename="$(find sensors_demos_gazebo)/meshes/utm30.dae" scale="1 1 1"/>
       </geometry>
     </collision>
@@ -23,5 +23,5 @@
       <origin xyz="0 0 0.0" rpy="1.57 0 0"/>
       <geometry>
-          <mesh filename="package://sensors_demos_gazebo/meshes/utm30.dae" scale="1 1 1"/>
+	  <mesh filename="$(find sensors_demos_gazebo)/meshes/utm30.dae" scale="1 1 1"/>
       </geometry>
       <material name="orange"/>
@@ -64,9 +64,13 @@
             </noise>
         </ray>
+     </sensor>
+     </gazebo>
+  <gazebo>
+   <sensor>
         <plugin name="gazebo_ros_head_hokuyo_controller" filename="libgazebo_ros_laser.so">
             <topicName>/head/utm30/laser/scan</topicName>
             <frameName>hokuyo_link</frameName>
-        </plugin>
-        </sensor>
-    </gazebo>
+    	</plugin>
+    </sensor>
+  </gazebo>
 </robot>

File: urdf/kinect.urdf.xacro (robot description, xacro)
@@ -17,5 +17,5 @@
       <origin xyz="0 0 0.1" rpy="0 0 0"/>
       <geometry>
-          <mesh filename="package://sensors_demos_gazebo/meshes/kinect.dae" scale="0.001 0.001 0.001"/>
+	<mesh filename="$(find sensors_demos_gazebo)/meshes/kinect.dae" scale="0.001 0.001 0.001" />
       </geometry>
     </collision>
@@ -23,5 +23,5 @@
       <origin xyz="0 0 0.1" rpy="0 0 0"/>
       <geometry>
-          <mesh filename="package://sensors_demos_gazebo/meshes/kinect.dae" scale="0.001 0.001 0.001"/>
+         <mesh filename="$(find sensors_demos_gazebo)/meshes/kinect.dae" scale="0.001 0.001 0.001" />
       </geometry>
       <material name="orange"/>
@@ -55,10 +55,10 @@
     <gazebo reference="kinect_optical_link">
     <sensor type="depth" name="kinect_depth_sensor">
-        <always_on>true</always_on>
+        <always_on>0</always_on>
+	<update_rate>1</update_rate>
         <horizontal_fov> ${91.2*3.14/180} </horizontal_fov>
         <vertical_fov> ${65.5*3.14/180} </vertical_fov>
         <diagonal_fov> ${100.6*3.14/180} </diagonal_fov>
-        <update_rate>6.0</update_rate>
-        <camera>
+        <camera name="kinect">
           <image>
             <format>R8G8B8</format>
@@ -76,5 +76,6 @@
           </noise>
         </camera>
-        <plugin name="kinect_frame_controller" filename="libgazebo_ros_openni_kinect.so">
+        <plugin name="kinect_frame_controller" filename="libgazebo_ros_camera.so">
+	   <camera_name>kinect</camera_name>
           <alwaysOn>true</alwaysOn>
           <updateRate>6.0</updateRate>
@@ -89,5 +90,5 @@
           <rangeMax>8.0</rangeMax>
         </plugin>
-      </sensor>
-  </gazebo>
+	</sensor>
+	</gazebo>
 </robot>

Commit message: Migration to ROS2, fixes

File: urdf/hokuyo.urdf.xacro (robot description, xacro)
@@ -1,75 +1,71 @@
 <?xml version="1.0"?>
 <robot name="sensor" xmlns:xacro="http://www.ros.org/wiki/xacro">
-      <xacro:property name="height1" value="1.2" />
-  <xacro:property name="height2" value="0.5" />
-  <xacro:property name="width" value="0.2" />
-  <xacro:property name="mass" value="0.1" />
- <!-- Used for fixing robot to Gazebo 'base_link' -->
-  <link name="world"/>
-  <joint name="fixed" type="fixed">
-    <parent link="world"/>
-    <child link="hokuyo_link"/>
-    <origin xyz="0 0 0.1" rpy="0 0 0"/>
-  </joint>
-  <!-- Hokuyo Link -->
-  <link name="hokuyo_link">
-    <collision>
-      <origin xyz="0 0 0.0" rpy="1.57 0 0"/>
-      <geometry>
-	  <mesh filename="$(find sensors_demos_gazebo)/meshes/utm30.dae" scale="1 1 1"/>
-      </geometry>
-    </collision>
-    <visual>
-      <origin xyz="0 0 0.0" rpy="1.57 0 0"/>
-      <geometry>
-	  <mesh filename="$(find sensors_demos_gazebo)/meshes/utm30.dae" scale="1 1 1"/>
-      </geometry>
-      <material name="orange"/>
-    </visual>
-    <inertial>
-      <origin xyz="0 0 0" rpy="0 0 0"/>
-      <mass value="${mass}"/>
-      <inertia
-	  ixx="${mass}" ixy="0.0" ixz="0.0"
-	  iyy="${mass}" iyz="0.0"
-	  izz="${mass}"/>
-    </inertial>
-  </link>
-  <material name="orange">
-    <color rgba="${255/255} ${108/255} ${10/255} 1.0"/>
-  </material>
-    <gazebo reference="hokuyo_link">
-        <sensor type="ray" name="head_hokuyo_sensor">
-        <pose>0 0 0.05 0 0 0</pose>
-        <visualize>true</visualize>
-        <update_rate>40</update_rate>
-        <ray>
-            <scan>
-            <horizontal>
-                <samples>720</samples>
-                <resolution>1</resolution>
-                <min_angle>-1.570796</min_angle>
-                <max_angle>1.570796</max_angle>
-            </horizontal>
-            </scan>
-            <range>
-            <min>0.10</min>
-            <max>30.0</max>
-            <resolution>0.01</resolution>
-            </range>
-            <noise>
-            <type>gaussian</type>
-            <mean>0.0</mean>
-            <stddev>0.01</stddev>
-            </noise>
-        </ray>
-        <plugin name="gazebo_ros_head_hokuyo_controller" filename="libgazebo_ros_ray_sensor.so">
-            <ros>
-               <remapping>~/out:=/hokuyo/scan</remapping>
-            </ros>
-            <frameName>hokuyo_link</frameName>
-            <output_type>sensor_msgs/LaserScan</output_type>
-    	</plugin>
-    </sensor>
-  </gazebo>
+    <xacro:property name="sensor_name" value="hokuyo" />
+    <xacro:property name="mass" value="0.1" />
+    <!-- Used for fixing robot to Gazebo 'base_link' -->
+    <link name="world"/>
+    <joint name="fixed" type="fixed">
+        <parent link="world"/>
+        <child link="${sensor_name}_link"/>
+        <origin xyz="0 0 0.1" rpy="0 0 0"/>
+    </joint>
+    <!-- Hokuyo Link -->
+    <link name="${sensor_name}_link">
+        <collision>
+            <origin xyz="0 0 0.0" rpy="1.57 0 0"/>
+            <geometry>
+                <mesh filename="$(find sensors_demos_gazebo)/meshes/utm30.dae" scale="1 1 1"/>
+            </geometry>
+        </collision>
+        <visual>
+            <origin xyz="0 0 0.0" rpy="1.57 0 0"/>
+            <geometry>
+                <mesh filename="$(find sensors_demos_gazebo)/meshes/utm30.dae" scale="1 1 1"/>
+            </geometry>
+            <material name="orange"/>
+        </visual>
+        <inertial>
+            <origin xyz="0 0 0" rpy="0 0 0"/>
+            <mass value="${mass}"/>
+            <inertia ixx="${mass}" ixy="0.0" ixz="0.0" iyy="${mass}" iyz="0.0" izz="${mass}"/>
+        </inertial>
+    </link>
+    <material name="orange">
+        <color rgba="${255/255} ${108/255} ${10/255} 1.0"/>
+    </material>
+    <gazebo reference="${sensor_name}_link">
+        <sensor type="ray" name="head_${sensor_name}_sensor">
+            <pose>0 0 0.05 0 0 0</pose>
+            <visualize>true</visualize>
+            <update_rate>40</update_rate>
+            <ray>
+                <scan>
+                    <horizontal>
+                        <samples>720</samples>
+                        <resolution>1</resolution>
+                        <min_angle>-1.570796</min_angle>
+                        <max_angle>1.570796</max_angle>
+                    </horizontal>
+                </scan>
+                <range>
+                    <min>0.10</min>
+                    <max>30.0</max>
+                    <resolution>0.01</resolution>
+                </range>
+                <noise>
+                    <type>gaussian</type>
+                    <mean>0.0</mean>
+                    <stddev>0.01</stddev>
+                </noise>
+            </ray>
+            <plugin name="gazebo_ros_head_${sensor_name}_controller" filename="libgazebo_ros_ray_sensor.so">
+                <ros>
+                    <namespace>/${sensor_name}</namespace>
+                    <remapping>~/out:=scan</remapping>
+                </ros>
+                <!-- <frame_name> ommited, will default to hokuo_link -->
+                <output_type>sensor_msgs/LaserScan</output_type>
+            </plugin>
+        </sensor>
+    </gazebo>
 </robot>
